File: daughterboard-supply.sch (KiCad schematic (older format))
At the start: 8 parts

Commit message: Added power connectors
Parts:
- C?: footprint nuc-compute-cluster-power-breakout-footprints:0402-cap -> antmicro-footprints:0402-cap; symbol nuc-compute-cluster-power-breakout:C_100n_0402 -> antmicroCapacitors0402:C_100n_0402
- C? (x2): footprint nuc-compute-cluster-power-breakout-footprints:0603-cap -> antmicro-footprints:0603-cap; symbol nuc-compute-cluster-power-breakout:C_22u_0603 -> antmicroCapacitors0603:C_22u_0603
- C?: footprint nuc-compute-cluster-power-breakout-footprints:0603-cap -> antmicro-footprints:0603-cap; symbol nuc-compute-cluster-power-breakout:C_10u_16V_0603 -> antmicroCapacitors0603:C_10u_16V_0603
- L?: footprint nuc-compute-cluster-power-breakout-footprints:WE_74437336033 -> antmicro-footprints:WE_74437336033; symbol nuc-compute-cluster-power-breakout:74437336033 -> antmicroFixedInductors:74437336033
- R?: footprint nuc-compute-cluster-power-breakout-footprints:0402-res -> antmicro-footprints:0402-res; symbol nuc-compute-cluster-power-breakout:R_10k_0402 -> antmicroResistors0402:R_10k_0402
- R?: footprint nuc-compute-cluster-power-breakout-footprints:0402-res -> antmicro-footprints:0402-res; symbol nuc-compute-cluster-power-breakout:R_52k3_0402 -> antmicroResistors0402:R_52k3_0402
- U?: footprint nuc-compute-cluster-power-breakout-footprints:TSOT23-6 -> antmicro-footprints:TSOT23-6; symbol nuc-compute-cluster-power-breakout:AP62301WU-7 -> antmicroDCDCConverters:AP62301WU-7
Changed lines of the file:
@@
 VCC12V0
 $Comp
-L nuc-compute-cluster-power-breakout:AP62301WU-7 U?
+L antmicroDCDCConverters:AP62301WU-7 U?
 U 1 1 6251678C
 P 3300 1750
@@
 F 0 "U?" H 3300 2215 50  0000 C CNN
 F 1 "AP62301WU-7" H 3300 2124 50  0000 C CNN
-F 2 "nuc-compute-cluster-power-breakout-footprints:TSOT23-6" H 3250 1100 50  0001 C CNN
+F 2 "antmicro-footprints:TSOT23-6" H 3250 1100 50  0001 C CNN
 F 3 "https://www.diodes.com/assets/Datasheets/AP62300_AP62301_AP62300T.pdf" H 3250 1400 50  0001 C CNN
 F 4 "AP62301WU-7" H 3250 1200 50  0001 C CNN "MPN"
@@
 $EndComp
 $Comp
-L nuc-compute-cluster-power-breakout:74437336033 L?
+L antmicroFixedInductors:74437336033 L?
 U 1 1 62516797
 P 4450 1550
@@
 F 0 "L?" H 4450 1855 60  0000 C CNN
 F 1 "74437336033" H 4450 1749 60  0000 C CNN
-F 2 "nuc-compute-cluster-power-breakout-footprints:WE_74437336033" H 5275 1900 60  0001 C CNN
+F 2 "antmicro-footprints:WE_74437336033" H 5275 1900 60  0001 C CNN
 F 3 "https://www.we-online.com/catalog/datasheet/74437336033.pdf" H 4505 1580 60  0001 C CNN
 F 4 "Wurth Elektronik" H 4750 2350 50  0001 C CNN "Manufacturer"
@@
 $EndComp
 $Comp
-L nuc-compute-cluster-power-breakout:C_100n_0402 C?
+L antmicroCapacitors0402:C_100n_0402 C?
 U 1 1 625167A0
 P 3950 1750
@@
 F 0 "C?" V 3850 1900 60  0000 C CNN
 F 1 "C_100n_0402" H 3950 1600 60  0001 C CNN
-F 2 "nuc-compute-cluster-power-breakout-footprints:0402-cap" H 4150 1950 60  0001 L CNN
+F 2 "antmicro-footprints:0402-cap" H 4150 1950 60  0001 L CNN
 F 3 "" H 3950 1750 50  0001 C CNN
 F 4 "Murata" H 4150 2150 60  0001 L CNN "Manufacturer"
@@
 	3700 1950 4700 1950
 $Comp
-L nuc-compute-cluster-power-breakout:GND #PWR?
+L power:GND #PWR?
 U 1 1 625167B6
 P 4700 2400
@@
 	4700 2400 4700 2300
 $Comp
-L nuc-compute-cluster-power-breakout:GND #PWR?
+L power:GND #PWR?
 U 1 1 625167CB
 P 2700 2400
@@
 	2700 1950 2900 1950
 $Comp
-L nuc-compute-cluster-power-breakout:C_22u_0603 C?
+L antmicroCapacitors0603:C_22u_0603 C?
 U 1 1 625167DF
 P 5150 1950
@@
 F 0 "C?" H 5265 1995 60  0000 L CNN
 F 1 "C_22u_0603" H 5150 1800 60  0001 C CNN
-F 2 "nuc-compute-cluster-power-breakout-footprints:0603-cap" H 5350 2150 60  0001 L CNN
+F 2 "antmicro-footprints:0603-cap" H 5350 2150 60  0001 L CNN
 F 3 "" H 5150 1950 50  0001 C CNN
 F 4 "MURATA" H 5350 2350 60  0001 L CNN "Manufacturer"
@@
 $EndComp
 $Comp
-L nuc-compute-cluster-power-breakout:C_22u_0603 C?
+L antmicroCapacitors0603:C_22u_0603 C?
 U 1 1 625167E8
 P 5500 1950
@@
 F 0 "C?" H 5615 1995 60  0000 L CNN
 F 1 "C_22u_0603" H 5500 1800 60  0001 C CNN
-F 2 "nuc-compute-cluster-power-breakout-footprints:0603-cap" H 5700 2150 60  0001 L CNN
+F 2 "antmicro-footprints:0603-cap" H 5700 2150 60  0001 L CNN
 F 3 "" H 5500 1950 50  0001 C CNN
 F 4 "MURATA" H 5700 2350 60  0001 L CNN "Manufacturer"
@@
 	2350 1550 2900 1550
 $Comp
-L nuc-compute-cluster-power-breakout:GND #PWR?
+L power:GND #PWR?
 U 1 1 625167F0
 P 2350 2400
@@
 	5150 1550 5500 1550
 $Comp
-L nuc-compute-cluster-power-breakout:GND #PWR?
+L power:GND #PWR?
 U 1 1 625167FD
 P 5150 2400
@@
 $EndComp
 $Comp
-L nuc-compute-cluster-power-breakout:GND #PWR?
+L power:GND #PWR?
 U 1 1 62516803
 P 5500 2400
@@
 Connection ~ 5500 1550
 $Comp
-L nuc-compute-cluster-power-breakout:C_10u_16V_0603 C?
+L antmicroCapacitors0603:C_10u_16V_0603 C?
 U 1 1 6252106D
 P 2350 2000
 F 0 "C?" H 2150 2100 60  0000 L CNN
 F 1 "C_10u_16V_0603" H 2350 1850 60  0001 C CNN
-F 2 "nuc-compute-cluster-power-breakout-footprints:0603-cap" H 2550 2200 60  0001 L CNN
+F 2 "antmicro-footprints:0603-cap" H 2550 2200 60  0001 L CNN
 F 3 "" H 2350 2000 50  0001 C CNN
 F 4 "MURATA" H 2550 2400 60  0001 L CNN "Manufacturer"
@@
 $EndComp
 $Comp
-L nuc-compute-cluster-power-breakout:R_10k_0402 R?
+L antmicroResistors0402:R_10k_0402 R?
 U 1 1 625167BF
 P 4700 2150
@@
 F 0 "R?" V 4655 2220 60  0000 L CNN
 F 1 "R_10k_0402" H 4700 2000 60  0001 C CNN
-F 2 "nuc-compute-cluster-power-breakout-footprints:0402-res" H 4900 2350 60  0001 L CNN
+F 2 "antmicro-footprints:0402-res" H 4900 2350 60  0001 L CNN
 F 3 "" H 4700 2150 50  0001 C CNN
 F 4 "VISHAY" H 4900 2550 60  0001 L CNN "Manufacturer"
@@
 $EndComp
 $Comp
-L nuc-compute-cluster-power-breakout:R_52k3_0402 R?
+L antmicroResistors0402:R_52k3_0402 R?
 U 1 1 6252687B
 P 4700 1750
 F 0 "R?" V 4655 1820 60  0000 L CNN
 F 1 "R_52k3_0402" H 4700 1600 60  0001 C CNN
-F 2 "nuc-compute-cluster-power-breakout-footprints:0402-res" H 4900 1950 60  0001 L CNN
+F 2 "antmicro-footprints:0402-res" H 4900 1950 60  0001 L CNN
 F 3 "" H 4700 1750 50  0001 C CNN
 F 4 "Panasonic" H 4900 2150 60  0001 L CNN "Manufacturer"

Commit message: loclib
Parts:
- C?: footprint antmicro-footprints:0402-cap -> nuc-compute-cluster-power-breakout-footprints:0402-cap; symbol antmicroCapacitors0402:C_100n_0402 -> nuc-compute-cluster-power-breakout:C_100n_0402
- C? (x2): footprint antmicro-footprints:0603-cap -> nuc-compute-cluster-power-breakout-footprints:0603-cap; symbol antmicroCapacitors0603:C_22u_0603 -> nuc-compute-cluster-power-breakout:C_22u_0603
- C?: footprint antmicro-footprints:0603-cap -> nuc-compute-cluster-power-breakout-footprints:0603-cap; symbol antmicroCapacitors0603:C_10u_16V_0603 -> nuc-compute-cluster-power-breakout:C_10u_16V_0603
- L?: footprint antmicro-footprints:WE_74437336033 -> nuc-compute-cluster-power-breakout-footprints:WE_74437336033; symbol antmicroFixedInductors:74437336033 -> nuc-compute-cluster-power-breakout:74437336033
- R?: footprint antmicro-footprints:0402-res -> nuc-compute-cluster-power-breakout-footprints:0402-res; symbol antmicroResistors0402:R_10k_0402 -> nuc-compute-cluster-power-breakout:R_10k_0402
- R?: footprint antmicro-footprints:0402-res -> nuc-compute-cluster-power-breakout-footprints:0402-res; symbol antmicroResistors0402:R_52k3_0402 -> nuc-compute-cluster-power-breakout:R_52k3_0402
- U?: footprint antmicro-footprints:TSOT23-6 -> nuc-compute-cluster-power-breakout-footprints:TSOT23-6; symbol antmicroDCDCConverters:AP62301WU-7 -> nuc-compute-cluster-power-breakout:AP62301WU-7
Changed lines of the file:
@@
 VCC12V0
 $Comp
-L antmicroDCDCConverters:AP62301WU-7 U?
+L nuc-compute-cluster-power-breakout:AP62301WU-7 U?
 U 1 1 6251678C
 P 3300 1750
@@
 F 0 "U?" H 3300 2215 50  0000 C CNN
 F 1 "AP62301WU-7" H 3300 2124 50  0000 C CNN
-F 2 "antmicro-footprints:TSOT23-6" H 3250 1100 50  0001 C CNN
+F 2 "nuc-compute-cluster-power-breakout-footprints:TSOT23-6" H 3250 1100 50  0001 C CNN
 F 3 "https://www.diodes.com/assets/Datasheets/AP62300_AP62301_AP62300T.pdf" H 3250 1400 50  0001 C CNN
 F 4 "AP62301WU-7" H 3250 1200 50  0001 C CNN "MPN"
@@
 $EndComp
 $Comp
-L antmicroFixedInductors:74437336033 L?
+L nuc-compute-cluster-power-breakout:74437336033 L?
 U 1 1 62516797
 P 4450 1550
@@
 F 0 "L?" H 4450 1855 60  0000 C CNN
 F 1 "74437336033" H 4450 1749 60  0000 C CNN
-F 2 "antmicro-footprints:WE_74437336033" H 5275 1900 60  0001 C CNN
+F 2 "nuc-compute-cluster-power-breakout-footprints:WE_74437336033" H 5275 1900 60  0001 C CNN
 F 3 "https://www.we-online.com/catalog/datasheet/74437336033.pdf" H 4505 1580 60  0001 C CNN
 F 4 "Wurth Elektronik" H 4750 2350 50  0001 C CNN "Manufacturer"
@@
 $EndComp
 $Comp
-L antmicroCapacitors0402:C_100n_0402 C?
+L nuc-compute-cluster-power-breakout:C_100n_0402 C?
 U 1 1 625167A0
 P 3950 1750
@@
 F 0 "C?" V 3850 1900 60  0000 C CNN
 F 1 "C_100n_0402" H 3950 1600 60  0001 C CNN
-F 2 "antmicro-footprints:0402-cap" H 4150 1950 60  0001 L CNN
+F 2 "nuc-compute-cluster-power-breakout-footprints:0402-cap" H 4150 1950 60  0001 L CNN
 F 3 "" H 3950 1750 50  0001 C CNN
 F 4 "Murata" H 4150 2150 60  0001 L CNN "Manufacturer"
@@
 	3700 1950 4700 1950
 $Comp
-L power:GND #PWR?
+L nuc-compute-cluster-power-breakout:GND #PWR?
 U 1 1 625167B6
 P 4700 2400
@@
 	4700 2400 4700 2300
 $Comp
-L power:GND #PWR?
+L nuc-compute-cluster-power-breakout:GND #PWR?
 U 1 1 625167CB
 P 2700 2400
@@
 	2700 1950 2900 1950
 $Comp
-L antmicroCapacitors0603:C_22u_0603 C?
+L nuc-compute-cluster-power-breakout:C_22u_0603 C?
 U 1 1 625167DF
 P 5150 1950
@@
 F 0 "C?" H 5265 1995 60  0000 L CNN
 F 1 "C_22u_0603" H 5150 1800 60  0001 C CNN
-F 2 "antmicro-footprints:0603-cap" H 5350 2150 60  0001 L CNN
+F 2 "nuc-compute-cluster-power-breakout-footprints:0603-cap" H 5350 2150 60  0001 L CNN
 F 3 "" H 5150 1950 50  0001 C CNN
 F 4 "MURATA" H 5350 2350 60  0001 L CNN "Manufacturer"
@@
 $EndComp
 $Comp
-L antmicroCapacitors0603:C_22u_0603 C?
+L nuc-compute-cluster-power-breakout:C_22u_0603 C?
 U 1 1 625167E8
 P 5500 1950
@@
 F 0 "C?" H 5615 1995 60  0000 L CNN
 F 1 "C_22u_0603" H 5500 1800 60  0001 C CNN
-F 2 "antmicro-footprints:0603-cap" H 5700 2150 60  0001 L CNN
+F 2 "nuc-compute-cluster-power-breakout-footprints:0603-cap" H 5700 2150 60  0001 L CNN
 F 3 "" H 5500 1950 50  0001 C CNN
 F 4 "MURATA" H 5700 2350 60  0001 L CNN "Manufacturer"
@@
 	2350 1550 2900 1550
 $Comp
-L power:GND #PWR?
+L nuc-compute-cluster-power-breakout:GND #PWR?
 U 1 1 625167F0
 P 2350 2400
@@
 	5150 1550 5500 1550
 $Comp
-L power:GND #PWR?
+L nuc-compute-cluster-power-breakout:GND #PWR?
 U 1 1 625167FD
 P 5150 2400
@@
 $EndComp
 $Comp
-L power:GND #PWR?
+L nuc-compute-cluster-power-breakout:GND #PWR?
 U 1 1 62516803
 P 5500 2400
@@
 Connection ~ 5500 1550
 $Comp
-L antmicroCapacitors0603:C_10u_16V_0603 C?
+L nuc-compute-cluster-power-breakout:C_10u_16V_0603 C?
 U 1 1 6252106D
 P 2350 2000
 F 0 "C?" H 2150 2100 60  0000 L CNN
 F 1 "C_10u_16V_0603" H 2350 1850 60  0001 C CNN
-F 2 "antmicro-footprints:0603-cap" H 2550 2200 60  0001 L CNN
+F 2 "nuc-compute-cluster-power-breakout-footprints:0603-cap" H 2550 2200 60  0001 L CNN
 F 3 "" H 2350 2000 50  0001 C CNN
 F 4 "MURATA" H 2550 2400 60  0001 L CNN "Manufacturer"
@@
 $EndComp
 $Comp
-L antmicroResistors0402:R_10k_0402 R?
+L nuc-compute-cluster-power-breakout:R_10k_0402 R?
 U 1 1 625167BF
 P 4700 2150
@@
 F 0 "R?" V 4655 2220 60  0000 L CNN
 F 1 "R_10k_0402" H 4700 2000 60  0001 C CNN
-F 2 "antmicro-footprints:0402-res" H 4900 2350 60  0001 L CNN
+F 2 "nuc-compute-cluster-power-breakout-footprints:0402-res" H 4900 2350 60  0001 L CNN
 F 3 "" H 4700 2150 50  0001 C CNN
 F 4 "VISHAY" H 4900 2550 60  0001 L CNN "Manufacturer"
@@
 $EndComp
 $Comp
-L antmicroResistors0402:R_52k3_0402 R?
+L nuc-compute-cluster-power-breakout:R_52k3_0402 R?
 U 1 1 6252687B
 P 4700 1750
 F 0 "R?" V 4655 1820 60  0000 L CNN
 F 1 "R_52k3_0402" H 4700 1600 60  0001 C CNN
-F 2 "antmicro-footprints:0402-res" H 4900 1950 60  0001 L CNN
+F 2 "nuc-compute-cluster-power-breakout-footprints:0402-res" H 4900 1950 60  0001 L CNN
 F 3 "" H 4700 1750 50  0001 C CNN
 F 4 "Panasonic" H 4900 2150 60  0001 L CNN "Manufacturer"
