File: pow-cycl-curr-meas.sch (KiCad schematic (older format))
At the start: 46 parts, among them Q1 SQS401EN-T1_BE3, Q10 SSM3K15ACT, Q2 SQS401EN-T1_BE3, Q3 SSM3K15ACT, Q4 SSM3K15ACT, Q5 SQS401EN-T1_BE3, Q6 SSM3K15ACT, Q7 SQS401EN-T1_BE3, Q8 SQS401EN-T1_BE3, Q9 SSM3K15ACT, U10 TCA9534, U11 TMCS1100A2-Q1, U12 TMCS1100A2-Q1, U13 TMCS1100A2-Q1, U14 ADS7828, U8 TMCS1100A2-Q1, U9 TMCS1100A2-Q1

Commit message: Loclib update
Parts:
- C21, C23, C28, C29, C30, C31, C32: footprint antmicro-footprints:0402-cap -> nuc-compute-cluster-power-breakout-footprints:0402-cap; symbol antmicroCapacitors0402:C_100n_0402 -> nuc-compute-cluster-power-breakout:C_100n_0402
- C22: footprint antmicro-footprints:0402-cap -> nuc-compute-cluster-power-breakout-footprints:0402-cap; symbol antmicroCapacitors0402:C_1u_0402 -> nuc-compute-cluster-power-breakout:C_1u_0402
- Q1, Q2, Q5, Q7, Q8: footprint antmicro-footprints:Vishay_PowerPAK_1212-8_Single -> nuc-compute-cluster-power-breakout-footprints:Vishay_PowerPAK_1212-8_Single; symbol antmicroTransistorsFETsMOSFETsSingle:SQS401EN-T1_BE3 -> nuc-compute-cluster-power-breakout:SQS401EN-T1_BE3
- Q10, Q3, Q4, Q6, Q9: footprint antmicro-footprints:SSM3K15ACT -> nuc-compute-cluster-power-breakout-footprints:SSM3K15ACT; symbol antmicroTransistorsFETsMOSFETsSingle:SSM3K15ACT -> nuc-compute-cluster-power-breakout:SSM3K15ACT
- R13, R14, R15, R16, R17, R18, R30, R31, R32, R33: footprint antmicro-footprints:0402-res -> nuc-compute-cluster-power-breakout-footprints:0402-res; symbol antmicroResistors0402:R_0R_0402 -> nuc-compute-cluster-power-breakout:R_0R_0402
- R19, R22, R23, R25, R28, R29: footprint antmicro-footprints:0402-res -> nuc-compute-cluster-power-breakout-footprints:0402-res; symbol antmicroResistors0402:R_4k7_0402 -> nuc-compute-cluster-power-breakout:R_4k7_0402
- R20, R21, R24, R26, R27: footprint antmicro-footprints:0402-res -> nuc-compute-cluster-power-breakout-footprints:0402-res; symbol antmicroResistors0402:R_10k_0402 -> nuc-compute-cluster-power-breakout:R_10k_0402
- U10: footprint antmicro-footprints:TSSOP-16 -> nuc-compute-cluster-power-breakout-footprints:TSSOP-16; symbol antmicroInterfaceIOExpanders:TCA9534 -> nuc-compute-cluster-power-breakout:TCA9534
- U11, U12, U13, U8, U9: footprint antmicro-footprints:SOIC-8_W3.9mm -> nuc-compute-cluster-power-breakout-footprints:SOIC-8_W3.9mm; symbol antmicroSensorsTransducersAccessories:TMCS1100A2-Q1 -> nuc-compute-cluster-power-breakout:TMCS1100A2-Q1
- U14: footprint Package_SO:TSSOP-16_4.4x5mm_P0.65mm -> nuc-compute-cluster-power-breakout-footprints:TSSOP-16_4.4x5mm_P0.65mm; symbol antmicroDataAcquisitionAnalogtoDigitalConvertersADC:ADS7828 -> nuc-compute-cluster-power-breakout:ADS7828

Commit message: Add remarks on the schematic sheets
Other:
- note added: "REMARK: Missing symbol"
- note added: "TODO: Add \nDNP fields\nto proper \nresistors"
Changed lines of the file:
@@
 U 1 1 62306CCE
 P 9600 8050
-F 0 "R28" V 9550 7850 60  0000 L CNN
+F 0 "R28" V 9550 7800 60  0000 L CNN
 F 1 "R_4k7_0402" H 9600 7900 60  0001 C CNN
 F 2 "nuc-compute-cluster-power-breakout-footprints:0402-res" H 9800 8250 60  0001 L CNN
@@
 U 1 1 622E9590
 P 9700 6050
-F 0 "R29" V 9650 5850 60  0000 L CNN
+F 0 "R29" V 9650 5800 60  0000 L CNN
 F 1 "R_4k7_0402" H 9700 5900 60  0001 C CNN
 F 2 "nuc-compute-cluster-power-breakout-footprints:0402-res" H 9900 6250 60  0001 L CNN
@@
 U 1 1 622C8CBE
 P 7900 9850
-F 0 "R25" V 7850 9650 60  0000 L CNN
+F 0 "R25" V 7850 9600 60  0000 L CNN
 F 1 "R_4k7_0402" H 7900 9700 60  0001 C CNN
 F 2 "nuc-compute-cluster-power-breakout-footprints:0402-res" H 8100 10050 60  0001 L CNN
@@
 U 1 1 6228D8DD
 P 6100 6100
-F 0 "R22" V 6050 5900 60  0000 L CNN
+F 0 "R22" V 6050 5850 60  0000 L CNN
 F 1 "R_4k7_0402" H 6100 5950 60  0001 C CNN
 F 2 "nuc-compute-cluster-power-breakout-footprints:0402-res" H 6300 6300 60  0001 L CNN
@@
 U 1 1 622D4C0D
 P 6150 8100
-F 0 "R23" V 6100 7900 60  0000 L CNN
+F 0 "R23" V 6100 7850 60  0000 L CNN
 F 1 "R_4k7_0402" H 6150 7950 60  0001 C CNN
 F 2 "nuc-compute-cluster-power-breakout-footprints:0402-res" H 6350 8300 60  0001 L CNN
@@
 Wire Wire Line
 	10250 3050 10400 3050
+Text Notes 575  7675 0    79   ~ 0
+TODO: Add \nDNP fields\nto proper \nresistors
+Text Notes 14400 9150 0    79   ~ 0
+REMARK: Missing symbol
+Text Notes 12150 3225 0    79   ~ 0
+TODO: Add \nDNP fields\nto proper \nresistors
 $EndSCHEMATC

Commit message: Improvements after review
Parts:
- added TP_ADC1, TP_ADC2, TP_ADC3, TP_ADC4, TP_ADC5, TP_PC1, TP_PC2, TP_PC3, TP_PC4, TP_PC5: TP_SMD1MM, antmicro-footprints:Testpoint_smd_1mm, symbol antmicroTestPoints:TP_SMD1MM
- R13, R15, R30, R32: DNP (none) -> DNP
- R17: DNP (none) -> DNP`
Connections:
- wire segments 221 -> 231
Other:
- note added: "ADC inputs TPs"
- note added: "Key transistors' polarization TPs"
- note removed: "REMARK: Missing symbol"
- note removed: "TODO: Add \nDNP fields\nto proper \nresistors"
- moved on the sheet: C21, C22, C23, C28, C29, C30, C31, C32, R30, R31, R32, R33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

Commit message: Loclib performed
Parts:
- TP_ADC1, TP_ADC2, TP_ADC3, TP_ADC4, TP_ADC5, TP_PC1, TP_PC2, TP_PC3, TP_PC4, TP_PC5: footprint antmicro-footprints:Testpoint_smd_1mm -> nuc-compute-cluster-power-breakout-footprints:Testpoint_smd_1mm; symbol antmicroTestPoints:TP_SMD1MM -> nuc-compute-cluster-power-breakout:TP_SMD1MM
Changed lines of the file:
@@
 	9850 3100 10000 3100
 $Comp
-L antmicroTestPoints:TP_SMD1MM TP_PC1
+L nuc-compute-cluster-power-breakout:TP_SMD1MM TP_PC1
 U 1 1 624C9924
 P 14200 8100
 F 0 "TP_PC1" V 14200 8050 50  0000 R CNN
 F 1 "TP_SMD1MM" H 14200 8000 50  0001 C CNN
-F 2 "antmicro-footprints:Testpoint_smd_1mm" H 14400 8300 60  0001 L CNN
+F 2 "nuc-compute-cluster-power-breakout-footprints:Testpoint_smd_1mm" H 14400 8300 60  0001 L CNN
 F 3 "" H 14400 8400 60  0001 L CNN
 	1    14200 8100
@@
 $EndComp
 $Comp
-L antmicroTestPoints:TP_SMD1MM TP_PC2
+L nuc-compute-cluster-power-breakout:TP_SMD1MM TP_PC2
 U 1 1 624CC7E9
 P 14200 8200
 F 0 "TP_PC2" V 14200 8150 50  0000 R CNN
 F 1 "TP_SMD1MM" H 14200 8100 50  0001 C CNN
-F 2 "antmicro-footprints:Testpoint_smd_1mm" H 14400 8400 60  0001 L CNN
+F 2 "nuc-compute-cluster-power-breakout-footprints:Testpoint_smd_1mm" H 14400 8400 60  0001 L CNN
 F 3 "" H 14400 8500 60  0001 L CNN
 	1    14200 8200
@@
 $EndComp
 $Comp
-L antmicroTestPoints:TP_SMD1MM TP_PC3
+L nuc-compute-cluster-power-breakout:TP_SMD1MM TP_PC3
 U 1 1 624CC9BA
 P 14200 8300
 F 0 "TP_PC3" V 14200 8250 50  0000 R CNN
 F 1 "TP_SMD1MM" H 14200 8200 50  0001 C CNN
-F 2 "antmicro-footprints:Testpoint_smd_1mm" H 14400 8500 60  0001 L CNN
+F 2 "nuc-compute-cluster-power-breakout-footprints:Testpoint_smd_1mm" H 14400 8500 60  0001 L CNN
 F 3 "" H 14400 8600 60  0001 L CNN
 	1    14200 8300
@@
 $EndComp
 $Comp
-L antmicroTestPoints:TP_SMD1MM TP_PC4
+L nuc-compute-cluster-power-breakout:TP_SMD1MM TP_PC4
 U 1 1 624CCB06
 P 14200 8400
 F 0 "TP_PC4" V 14200 8350 50  0000 R CNN
 F 1 "TP_SMD1MM" H 14200 8300 50  0001 C CNN
-F 2 "antmicro-footprints:Testpoint_smd_1mm" H 14400 8600 60  0001 L CNN
+F 2 "nuc-compute-cluster-power-breakout-footprints:Testpoint_smd_1mm" H 14400 8600 60  0001 L CNN
 F 3 "" H 14400 8700 60  0001 L CNN
 	1    14200 8400
@@
 $EndComp
 $Comp
-L antmicroTestPoints:TP_SMD1MM TP_PC5
+L nuc-compute-cluster-power-breakout:TP_SMD1MM TP_PC5
 U 1 1 624CCCA3
 P 14200 8500
 F 0 "TP_PC5" V 14200 8450 50  0000 R CNN
 F 1 "TP_SMD1MM" H 14200 8400 50  0001 C CNN
-F 2 "antmicro-footprints:Testpoint_smd_1mm" H 14400 8700 60  0001 L CNN
+F 2 "nuc-compute-cluster-power-breakout-footprints:Testpoint_smd_1mm" H 14400 8700 60  0001 L CNN
 F 3 "" H 14400 8800 60  0001 L CNN
 	1    14200 8500
@@
 Key transistors' polarization TPs
 $Comp
-L antmicroTestPoints:TP_SMD1MM TP_ADC1
+L nuc-compute-cluster-power-breakout:TP_SMD1MM TP_ADC1
 U 1 1 625E59A0
 P 14400 3700
 F 0 "TP_ADC1" V 14400 3650 50  0000 R CNN
 F 1 "TP_SMD1MM" H 14400 3600 50  0001 C CNN
-F 2 "antmicro-footprints:Testpoint_smd_1mm" H 14600 3900 60  0001 L CNN
+F 2 "nuc-compute-cluster-power-breakout-footprints:Testpoint_smd_1mm" H 14600 3900 60  0001 L CNN
 F 3 "" H 14600 4000 60  0001 L CNN
 	1    14400 3700
@@
 $EndComp
 $Comp
-L antmicroTestPoints:TP_SMD1MM TP_ADC2
+L nuc-compute-cluster-power-breakout:TP_SMD1MM TP_ADC2
 U 1 1 625E6F51
 P 14400 3800
 F 0 "TP_ADC2" V 14400 3750 50  0000 R CNN
 F 1 "TP_SMD1MM" H 14400 3700 50  0001 C CNN
-F 2 "antmicro-footprints:Testpoint_smd_1mm" H 14600 4000 60  0001 L CNN
+F 2 "nuc-compute-cluster-power-breakout-footprints:Testpoint_smd_1mm" H 14600 4000 60  0001 L CNN
 F 3 "" H 14600 4100 60  0001 L CNN
 	1    14400 3800
@@
 $EndComp
 $Comp
-L antmicroTestPoints:TP_SMD1MM TP_ADC3
+L nuc-compute-cluster-power-breakout:TP_SMD1MM TP_ADC3
 U 1 1 625E7235
 P 14400 3900
 F 0 "TP_ADC3" V 14400 3850 50  0000 R CNN
 F 1 "TP_SMD1MM" H 14400 3800 50  0001 C CNN
-F 2 "antmicro-footprints:Testpoint_smd_1mm" H 14600 4100 60  0001 L CNN
+F 2 "nuc-compute-cluster-power-breakout-footprints:Testpoint_smd_1mm" H 14600 4100 60  0001 L CNN
 F 3 "" H 14600 4200 60  0001 L CNN
 	1    14400 3900
@@
 $EndComp
 $Comp
-L antmicroTestPoints:TP_SMD1MM TP_ADC4
+L nuc-compute-cluster-power-breakout:TP_SMD1MM TP_ADC4
 U 1 1 625E7421
 P 14400 4000
 F 0 "TP_ADC4" V 14400 3950 50  0000 R CNN
 F 1 "TP_SMD1MM" H 14400 3900 50  0001 C CNN
-F 2 "antmicro-footprints:Testpoint_smd_1mm" H 14600 4200 60  0001 L CNN
+F 2 "nuc-compute-cluster-power-breakout-footprints:Testpoint_smd_1mm" H 14600 4200 60  0001 L CNN
 F 3 "" H 14600 4300 60  0001 L CNN
 	1    14400 4000
@@
 $EndComp
 $Comp
-L antmicroTestPoints:TP_SMD1MM TP_ADC5
+L nuc-compute-cluster-power-breakout:TP_SMD1MM TP_ADC5
 U 1 1 625E7646
 P 14400 4100
 F 0 "TP_ADC5" V 14400 4050 50  0000 R CNN
 F 1 "TP_SMD1MM" H 14400 4000 50  0001 C CNN
-F 2 "antmicro-footprints:Testpoint_smd_1mm" H 14600 4300 60  0001 L CNN
+F 2 "nuc-compute-cluster-power-breakout-footprints:Testpoint_smd_1mm" H 14600 4300 60  0001 L CNN
 F 3 "" H 14600 4400 60  0001 L CNN
 	1    14400 4100

Commit message: Patches after 2nd revision
Parts:
- U14: footprint nuc-compute-cluster-power-breakout-footprints:TSSOP-16_4.4x5mm_P0.65mm -> antmicro-footprints:TSSOP-16_4.4x5mm_P0.65mm
Changed lines of the file:
@@
 F 0 "U14" H 10100 3350 50  0000 C CNN
 F 1 "ADS7828" H 10100 3250 50  0000 C CNN
-F 2 "nuc-compute-cluster-power-breakout-footprints:TSSOP-16_4.4x5mm_P0.65mm" H 11350 1900 50  0001 C CNN
+F 2 "antmicro-footprints:TSSOP-16_4.4x5mm_P0.65mm" H 11350 1900 50  0001 C CNN
 F 3 "http://www.ti.com/lit/ds/symlink/ads7828.pdf" H 10400 2600 50  0001 C CNN
 F 4 "ADS7828E/250 " H 10400 2600 50  0001 C CNN "MPN"

Commit message: Performed loclib
Parts:
- U14: footprint antmicro-footprints:TSSOP-16_4.4x5mm_P0.65mm -> nuc-compute-cluster-power-breakout-footprints:TSSOP-16_4.4x5mm_P0.65mm
Changed lines of the file:
@@
 F 0 "U14" H 10100 3350 50  0000 C CNN
 F 1 "ADS7828" H 10100 3250 50  0000 C CNN
-F 2 "antmicro-footprints:TSSOP-16_4.4x5mm_P0.65mm" H 11350 1900 50  0001 C CNN
+F 2 "nuc-compute-cluster-power-breakout-footprints:TSSOP-16_4.4x5mm_P0.65mm" H 11350 1900 50  0001 C CNN
 F 3 "http://www.ti.com/lit/ds/symlink/ads7828.pdf" H 10400 2600 50  0001 C CNN
 F 4 "ADS7828E/250 " H 10400 2600 50  0001 C CNN "MPN"
