File: nuc-compute-cluster-power-breakout.kicad_pcb (KiCad board)
At the start: 4 copper layers, 100 x 100 mm, 169 parts, among them J1 USB3106-30-0230-A, J10 10107844-002LF, J2 BM04B-SRSS-TB-LF-SN, J3 BM04B-SRSS-TB-LF-SN, J4 43045-1013, J5 430450812, J6 430450812, J7 430450812, J8 430450812, J9 430450812, Q1 SQS401EN-T1_BE3, Q10 SSM3K15ACT, Q11 BC856,215, Q2 SQS401EN-T1_BE3, Q3 SSM3K15ACT, Q4 SSM3K15ACT, Q5 SQS401EN-T1_BE3, Q6 SSM3K15ACT, Q7 SQS401EN-T1_BE3, Q8 SQS401EN-T1_BE3, Q9 SSM3K15ACT, U1 FT2232HL-REEL, U10 TCA9534, U11 TMCS1100A2-Q1, U12 TMCS1100A2-Q1, U13 TMCS1100A2-Q1, U14 ADS7828, U15 AP62301WU-7, U2 ISO1641, U3 NCP163ASN330T1G, U4 AP62301WU-7, U8 TMCS1100A2-Q1, U9 TMCS1100A2-Q1, Y1 KX-7_12,MHz

Commit message: Layout of power connectors
Parts:
- removed C23: C_100n_0402, nuc-compute-cluster-power-breakout-footprints:0402-cap
- added C37: C_100n_0402, nuc-compute-cluster-power-breakout-footprints:0402-cap, F.Cu at (149.9, 103.7)
- added FB4: BLM18AG601SN1D, nuc-compute-cluster-power-breakout-footprints:0603, F.Cu at (149.6, 105.0)
- C13: value C_3u3_0402 -> C_4u7_0402; footprint nuc-compute-cluster-power-breakout-footprints:0402-cap -> antmicro-footprints:0402-cap
- C14, C15: value C_4n7_0402 -> C_4u7_0402; footprint nuc-compute-cluster-power-breakout-footprints:0402-cap -> antmicro-footprints:0402-cap
- C19, C20: value C_1u_0402 -> C_4u7_0402; footprint nuc-compute-cluster-power-breakout-footprints:0402-cap -> antmicro-footprints:0402-cap
- J4: value 43045-1013 -> 39288080; footprint nuc-compute-cluster-power-breakout-footprints:43045-1013 -> antmicro-footprints:MOLEX_39288080
- J5, J6, J7, J8: value 430450812 -> 39288080; footprint nuc-compute-cluster-power-breakout-footprints:Molex-43045-0812 -> antmicro-footprints:MOLEX_39288080
- J9: value 430450812 -> 39281103; footprint nuc-compute-cluster-power-breakout-footprints:Molex-43045-0812 -> antmicro-footprints:MOLEX_39281103
- R1: value R_4k7_0402 -> R_1k_0402; footprint nuc-compute-cluster-power-breakout-footprints:0402-res -> antmicro-footprints:0402-res
- R2: value R_10k_0402 -> R_0R_0402; footprint nuc-compute-cluster-power-breakout-footprints:0402-res -> antmicro-footprints:0402-res
- moved J9 85.6 mm to (94.2, 78.9)
- moved R2 72.9 mm to (106.3, 81.0)
- moved J6 47.3 mm to (179.5, 74.7)
- moved R43 39.4 mm to (107.1, 96.0), turned to -90 degrees
- moved C34 39.0 mm to (104.6, 97.5), turned to 90 degrees
- moved R44 38.8 mm to (108.1, 96.0), turned to 90 degrees
- moved C36 37.5 mm to (103.0, 99.8), turned to 90 degrees
- moved C35 36.3 mm to (104.5, 99.8), turned to 90 degrees
- moved U4 35.4 mm to (107.1, 99.1), turned to 0 degrees
- moved C33 33.0 mm to (109.7, 99.8), turned to 90 degrees
- moved L1 30.1 mm to (106.0, 104.1), turned to 180 degrees
- moved 3V3 29.9 mm to (100.8, 105.3), turned to 90 degrees
- moved J5 29.0 mm to (145.2, 74.7)
- moved J7 23.1 mm to (128.2, 74.7)
- moved J4 19.9 mm to (111.2, 74.7), turned to 90 degrees
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Connections:
- J1 pad 4: Net-(J1-Pad4) -> unconnected-(J1-Pad4)
- J10 pad P19/20: Net-(J10-PadP19/20) -> unconnected-(J10-PadP19/20)
- J4 pad 5: VCC3V3 -> LOAD_1
- J4 pad 6: VCC12V0 -> LOAD_1
- J4 pad 7: VCC12V0 -> LOAD_1
- J4 pad 8: VCC5V0 -> LOAD_1
- J5 pad 1: LOAD_1 -> GND
- J5 pad 2: LOAD_1 -> GND
- J5 pad 3: LOAD_1 -> GND
- J5 pad 4: LOAD_1 -> GND
- J5 pad 5: GND -> LOAD_3
- J5 pad 6: GND -> LOAD_3
- J5 pad 7: GND -> LOAD_3
- J5 pad 8: GND -> LOAD_3
- J6 pad 1: LOAD_2 -> GND
- J6 pad 2: LOAD_2 -> GND
- J6 pad 3: LOAD_2 -> GND
- J6 pad 4: LOAD_2 -> GND
- J6 pad 5: GND -> LOAD_5
- J6 pad 6: GND -> LOAD_5
- J6 pad 7: GND -> LOAD_5
- J6 pad 8: GND -> LOAD_5
- J7 pad 1: LOAD_3 -> GND
- J7 pad 2: LOAD_3 -> GND
- J7 pad 3: LOAD_3 -> GND
- J7 pad 4: LOAD_3 -> GND
- J7 pad 5: GND -> LOAD_2
- J7 pad 6: GND -> LOAD_2
- J7 pad 7: GND -> LOAD_2
- J7 pad 8: GND -> LOAD_2
- J8 pad 1: LOAD_4 -> GND
- J8 pad 2: LOAD_4 -> GND
- J8 pad 3: LOAD_4 -> GND
- J8 pad 4: LOAD_4 -> GND
- J8 pad 5: GND -> LOAD_4
- J8 pad 6: GND -> LOAD_4
- J8 pad 7: GND -> LOAD_4
- J8 pad 8: GND -> LOAD_4
- J9 pad 1: LOAD_5 -> VCC3V3
- J9 pad 2: LOAD_5 -> GND
- J9 pad 3: LOAD_5 -> VCC5V0
- J9 pad 4: LOAD_5 -> VCC12V0
- J9 pad 5: GND -> VCC12V0
- J9 pad 6: GND -> VCC3V3
- J9 pad 8: GND -> Net-(J9-Pad8)
- R11 pad 2: SDA_FTDI -> SCL_FTDI
- R12 pad 2: SCL_FTDI -> SDA_FTDI
- R2 pad 1: /FTDI/FTDI_RST -> Net-(J9-Pad8)
- R2 pad 2: GNDD -> GND
- S1 pad 1: Net-(S1-Pad1) -> unconnected-(S1-Pad1)
- U1 pad 21: Net-(U1-Pad21) -> unconnected-(U1-Pad21)
- U1 pad 22: Net-(U1-Pad22) -> unconnected-(U1-Pad22)
- U1 pad 23: Net-(U1-Pad23) -> unconnected-(U1-Pad23)
- U1 pad 24: Net-(U1-Pad24) -> unconnected-(U1-Pad24)
- U1 pad 26: Net-(U1-Pad26) -> unconnected-(U1-Pad26)
- U1 pad 27: Net-(U1-Pad27) -> unconnected-(U1-Pad27)
- U1 pad 28: Net-(U1-Pad28) -> unconnected-(U1-Pad28)
- U1 pad 29: Net-(U1-Pad29) -> unconnected-(U1-Pad29)
- U1 pad 30: Net-(U1-Pad30) -> unconnected-(U1-Pad30)
- U1 pad 32: Net-(U1-Pad32) -> unconnected-(U1-Pad32)
- U1 pad 33: Net-(U1-Pad33) -> unconnected-(U1-Pad33)
- U1 pad 34: Net-(U1-Pad34) -> unconnected-(U1-Pad34)
- U1 pad 36: Net-(U1-Pad36) -> unconnected-(U1-Pad36)
- U1 pad 38: Net-(U1-Pad38) -> unconnected-(U1-Pad38)
- U1 pad 39: Net-(U1-Pad39) -> unconnected-(U1-Pad39)
- U1 pad 40: Net-(U1-Pad40) -> unconnected-(U1-Pad40)
- U1 pad 41: Net-(U1-Pad41) -> unconnected-(U1-Pad41)
- U1 pad 43: Net-(U1-Pad43) -> unconnected-(U1-Pad43)
- U1 pad 44: Net-(U1-Pad44) -> unconnected-(U1-Pad44)
- U1 pad 45: Net-(U1-Pad45) -> unconnected-(U1-Pad45)
- U1 pad 46: Net-(U1-Pad46) -> unconnected-(U1-Pad46)
- U1 pad 48: Net-(U1-Pad48) -> unconnected-(U1-Pad48)
- U1 pad 52: Net-(U1-Pad52) -> unconnected-(U1-Pad52)
- U1 pad 53: Net-(U1-Pad53) -> unconnected-(U1-Pad53)
- U1 pad 54: Net-(U1-Pad54) -> unconnected-(U1-Pad54)
- U1 pad 55: Net-(U1-Pad55) -> unconnected-(U1-Pad55)
- U1 pad 57: Net-(U1-Pad57) -> unconnected-(U1-Pad57)
- U1 pad 58: Net-(U1-Pad58) -> unconnected-(U1-Pad58)
- U1 pad 59: Net-(U1-Pad59) -> unconnected-(U1-Pad59)
- U1 pad 60: Net-(U1-Pad60) -> unconnected-(U1-Pad60)
- U1 pad 61: Net-(U1-Pad61) -> unconnected-(U1-Pad61)
- U1 pad 62: Net-(U1-Pad62) -> unconnected-(U1-Pad62)
- U1 pad 63: Net-(U1-Pad63) -> unconnected-(U1-Pad63)
- U10 pad 10: Net-(U10-Pad10) -> unconnected-(U10-Pad10)
- U10 pad 11: Net-(U10-Pad11) -> unconnected-(U10-Pad11)
- U10 pad 12: Net-(U10-Pad12) -> unconnected-(U10-Pad12)
- U14 pad 10: VCC3V3 -> Net-(U14-Pad10)
- U14 pad 6: Net-(U14-Pad6) -> unconnected-(U14-Pad6)
- U14 pad 7: Net-(U14-Pad7) -> unconnected-(U14-Pad7)
- U14 pad 8: Net-(U14-Pad8) -> unconnected-(U14-Pad8)
- U15 pad 5: Net-(U15-Pad5) -> unconnected-(U15-Pad5)
- U4 pad 5: Net-(U4-Pad5) -> unconnected-(U4-Pad5)
Routing:
- net VCC3V3: track 157.6 -> 103.2 mm, vias 34 -> 33
- net VCC12V0: track 47.8 -> 19.1 mm, vias 171 -> 225
- net GNDD: track 34.3 -> 13.9 mm, vias 7 -> 10
- net Net-(J9-Pad8): track 0.00 -> 15.0 mm
- net /Power Cycling & Current Measurement/PC_3: track 37.5 -> 27.0 mm, vias 3 -> 1
- net GND: track 56.9 -> 46.9 mm, vias 297 -> 364
- net /Power Cycling & Current Measurement/PC_4: track 23.0 -> 15.8 mm, vias 2 -> 0
- net /Power Cycling & Current Measurement/PC_1: track 59.3 -> 65.8 mm
- net /Power Cycling & Current Measurement/C_ADC4: track 25.1 -> 19.3 mm, vias 0 -> 2
- net SDA_FTDI: track 21.7 -> 26.2 mm
- net /Power Cycling & Current Measurement/C_ADC5: track 38.3 -> 34.5 mm, vias 0 -> 2
- net /Power Cycling & Current Measurement/PC_2: track 47.0 -> 43.4 mm, vias 2 -> 1
- net VCC5V0: track 13.7 -> 10.1 mm
- net Net-(U14-Pad10): track 0.00 -> 3.00 mm
- net /Power Cycling & Current Measurement/PC_5: track 33.0 -> 30.1 mm
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- added copper zone on In2.Cu, net GNDD
- added copper zone on In2.Cu, net VCC12V0

Commit message: Finished layout and fixed silkscreen
Parts:
- moved N2 13.8 mm to (108.7, 120.8)
- moved N1 7.05 mm to (101.8, 112.4)
Routing:
- net VCC12V0: track 19.1 -> 1.50 mm, vias 225 -> 227
- net GND: track 46.9 -> 30.0 mm, vias 364 -> 442
- net /Power Cycling & Current Measurement/C_ADC1: track 59.9 -> 57.5 mm
- net VCC3V3: track 103.2 -> 100.8 mm
- net Net-(J10-PadS24): track 11.5 -> 9.05 mm
- net Net-(J10-PadS23): track 11.5 -> 9.20 mm
- net SCL: track 59.6 -> 58.6 mm
- net /Power Cycling & Current Measurement/C_ADC2: track 43.0 -> 42.3 mm
- net /Power Cycling & Current Measurement/C_ADC3: track 29.1 -> 28.4 mm
- net /Power Cycling & Current Measurement/PC_3: track 27.0 -> 26.6 mm, vias 1 -> 0
- net GNDD: track 13.9 -> 13.6 mm, vias 10 -> 9
- net /Power Cycling & Current Measurement/PC_1: track 65.8 -> 65.7 mm, vias 3 -> 2
- net Net-(C25-Pad1): vias 1 -> 0
- net /Power Cycling & Current Measurement/PC_2: vias 1 -> 0
Other:
- board text added: "1"
- board text added: "2"
- board text added: "3"
- board text added: "4"
- board text added: "5"
- board text added: "ADC1"
- board text added: "ADC2"
- board text added: "ADC3"
- board text added: "ADC4"
- board text added: "ADC5"
- board text added: "PC"
