File: d1600e-psu-breakout-board.kicad_sch (KiCad schematic)
At the start: 69 parts, among them J1 4PIN-22-27-2041, J10 10107844-002LF, J11 4PIN-22-27-2041, J12 4PIN-22-27-2041, J13 4PIN-22-27-2041, J14 4PIN-22-27-2041, J2 BM04B-SRSS-TB-LF-SN, J3 BM04B-SRSS-TB-LF-SN, J4 39288080, J5 39288080, J6 39288080, J7 39288080, J8 39288080, Q11 BC856,215

Commit message: [#63472] Add OHP assets
Parts:
- removed J1, J11, J12, J13, J14: 4PIN-22-27-2041, antmicro-footprints:4PIN-22-27-2041, symbol antmicroRectangularConnectorsHeadersMalePins:4PIN-22-27-2041
- removed J4, J5, J6, J7, J8: 39288080, d1600e-psu-breakout-board-footprints:MOLEX_39288080, symbol d1600e-psu-breakout-board:39288080
- removed MP1, MP2, MP3, MP4: PCB_Mount_Hole_3mm_6mm_pad, d1600e-psu-breakout-board-footprints:mounting-hole-3.2mm, symbol d1600e-psu-breakout-board:PCB_Mount_Hole_3mm_6mm_pad
- removed N1: oshw_logo, d1600e-psu-breakout-board-footprints:OSHW-Logo_7.5x8mm_Mask, symbol d1600e-psu-breakout-board:oshw_logo
- removed N2: antmicro_logo, d1600e-psu-breakout-board-footprints:antmicro-logo_scaled_20mm_mask, symbol d1600e-psu-breakout-board:antmicro_logo
- removed Q11: BC856,215, d1600e-psu-breakout-board-footprints:SOT-23-3, symbol d1600e-psu-breakout-board:BC856,215
- removed S1: MSS3-V-T_R, d1600e-psu-breakout-board-footprints:Switch_Slide_MSS3, symbol d1600e-psu-breakout-board:MSS3-V-T_R
- added J1, J11, J12, J13, J14: Molex_KK_1x4_22-27-2041, antmicro-footprints:Conn_Molex_KK_1x4_22-27-2041, symbol antmicroWire2BoardConnectors:Molex_KK_1x4_22-27-2041
- added J4, J5, J6, J7, J8: Molex_Mini-Fit-Jr_2x4_39-28-8080, antmicro-footprints:MOLEX_39288080, symbol antmicroWire2BoardConnectors:Molex_Mini-Fit-Jr_2x4_39-28-8080
- added MP1, MP2, MP3, MP4: MP_Pad6mm_Drill3.2mm, antmicro-footprints:MP_Pad6mm_Drill3.2mm, symbol antmicroMechanicalParts:MP_Pad6mm_Drill3.2mm
- added Q11: BC856,215, antmicro-footprints:SOT-23-3, symbol antmicroTransistorsBipolarSingle:BC856,215
- added S1: SW_SPDT_PCM12SMTR, antmicro-footprints:PCM12SMTR, symbol antmicroSlideSwitches:SW_SPDT_PCM12SMTR
- D10, D11, D3, D4, D5, D6, D7, D8, D9: value LG_L29K-G2J1-24-Z -> LED_G_0603_LG_L29K-G2J1-24-Z; footprint d1600e-psu-breakout-board-footprints:LED_0603 -> antmicro-footprints:LED_0603_1608Metric_G; symbol d1600e-psu-breakout-board:LG_L29K-G2J1-24-Z -> antmicroLEDIndicationDiscrete:LED_G_0603_LG_L29K-G2J1-24-Z; Author (none) -> Antmicro; Color (none) -> Green; License (none) -> Apache-2.0; Manufacturer OSRAM Opto Semiconductors Inc. -> OSRAM
- D12, D13: footprint d1600e-psu-breakout-board-footprints:TPD2E009DRTR -> antmicro-footprints:TPD2E009DRTR; symbol d1600e-psu-breakout-board:PESD5V0S2BQA -> antmicroTVSDiodes:PESD5V0S2BQA; Author (none) -> Antmicro; License (none) -> Apache-2.0
- J10: value 10107844-002LF -> Socket_Amphenol_HPCE_2x17_10107844-002LF; footprint d1600e-psu-breakout-board-footprints:10107844-002LF -> antmicro-footprints:Socket_Amphenol_HPCE_2x17_10107844-002LF; symbol d1600e-psu-breakout-board:10107844-002LF -> antmicroEdgeConnectors:Socket_Amphenol_HPCE_2x17_10107844-002LF; Author (none) -> Antmicro; License (none) -> Apache-2.0
- J2: value BM04B-SRSS-TB-LF-SN -> JST_SH_1x4_BM04B-SRSS-TB-LF-SN; footprint d1600e-psu-breakout-board-footprints:BM04B-SRSS-TB-LF-SN -> antmicro-footprints:Conn_JST_SH_1x4_BM04B-SRSS-TB-LF-SN; symbol d1600e-psu-breakout-board:BM04B-SRSS-TB-LF-SN -> antmicroWire2BoardConnectors:JST_SH_1x4_BM04B-SRSS-TB-LF-SN; Author (none) -> Antmicro; License (none) -> Apache-2.0; Manufacturer JST -> JST Automotive Connectors; now not fitted; now left out of the parts list
- J3: value BM04B-SRSS-TB-LF-SN -> JST_SH_1x4_BM04B-SRSS-TB-LF-SN; footprint d1600e-psu-breakout-board-footprints:BM04B-SRSS-TB-LF-SN -> antmicro-footprints:Conn_JST_SH_1x4_BM04B-SRSS-TB-LF-SN; symbol d1600e-psu-breakout-board:BM04B-SRSS-TB-LF-SN -> antmicroWire2BoardConnectors:JST_SH_1x4_BM04B-SRSS-TB-LF-SN; Author (none) -> Antmicro; License (none) -> Apache-2.0; Manufacturer JST -> JST Automotive Connectors
- R10, R45, R9: footprint d1600e-psu-breakout-board-footprints:0402-res -> antmicro-footprints:R_0402_1005Metric; symbol d1600e-psu-breakout-board:R_0R_0402 -> antmicroResistors0402:R_0R_0402; Author (none) -> Antmicro; Current (none) -> 1A; License (none) -> Apache-2.0; Manufacturer PANASONIC -> Panasonic; now not fitted; now left out of the parts list
- R11, R12, R51, R52, R53: footprint d1600e-psu-breakout-board-footprints:0603-res -> antmicro-footprints:R_0603_1608Metric; symbol d1600e-psu-breakout-board:R_4k7_0603 -> antmicroResistors0603:R_4k7_0603; Author (none) -> Antmicro; License (none) -> Apache-2.0; Manufacturer BOURNS -> Bourns; Tolerance (none) -> 1%
- R40: footprint d1600e-psu-breakout-board-footprints:0402-res -> antmicro-footprints:R_0402_1005Metric; symbol d1600e-psu-breakout-board:R_10k_0402 -> antmicroResistors0402:R_10k_0402; Author (none) -> Antmicro; License (none) -> Apache-2.0; MPN CRCW040210K0FKEDHP -> CR0402-FX-1002GLF; Manufacturer VISHAY -> Bourns; Tolerance (none) -> 1%
- R41: footprint d1600e-psu-breakout-board-footprints:0402-res -> antmicro-footprints:R_0402_1005Metric; symbol d1600e-psu-breakout-board:R_680R_0402 -> antmicroResistors0402:R_680R_0402; Author (none) -> Antmicro; License (none) -> Apache-2.0; MPN 0402WGJ0681TCE -> CR0402-FX-6800GLF; Manufacturer ROYAL_OHM -> Bourns; Tolerance (none) -> 1%
- R54, R55: footprint d1600e-psu-breakout-board-footprints:0603-res -> antmicro-footprints:R_0603_1608Metric; symbol d1600e-psu-breakout-board:R_1k_0603 -> antmicroResistors0603:R_1k_0603; Author (none) -> Antmicro; License (none) -> Apache-2.0; MPN CR0603-JW-102ELF -> CR0603-FX-1001ELF; Manufacturer BOURNS -> Bourns; Tolerance (none) -> 1%
- R56: footprint d1600e-psu-breakout-board-footprints:0603-res -> antmicro-footprints:R_0603_1608Metric; symbol d1600e-psu-breakout-board:R_2k2_0603 -> antmicroResistors0603:R_2k2_0603; Author (none) -> Antmicro; License (none) -> Apache-2.0; MPN MCMR06X2201FTL -> CR0603-FX-2201ELF; Manufacturer MULTICOMP -> Bourns; Tolerance (none) -> 1%
- R71: now not fitted; now left out of the parts list
- TP_S1, TP_S10, TP_S11, TP_S12, TP_S16, TP_S17, TP_S18, TP_S19, TP_S2, TP_S20, TP_S21, TP_S22, TP_S23, TP_S24, TP_S3, TP_S4, TP_S5, TP_S6, TP_S7, TP_S8, TP_S9, TP_S_ON1: value TP_SMD1MM -> TP_1mm_SMD; footprint d1600e-psu-breakout-board-footprints:Testpoint_smd_1mm -> antmicro-footprints:TP_SMD_1mm; symbol d1600e-psu-breakout-board:TP_SMD1MM -> antmicroTestPoints:TP_1mm_SMD; Author (none) -> Antmicro; License (none) -> Apache-2.0; now left out of the parts list
Connections:
- net GND: now also D10.1 (C), D11.1 (C), D3.1 (C), D4.1 (C), D6.1 (C), D7.1 (C), D8.1 (C), D9.1 (C), J1.2, J1.3, J11.2, J11.3, J12.2, J12.3, J13.2, J13.3, J14.2, J14.3, J4.1, J4.2, J4.3, J4.4, J5.1, J5.2, J5.3, J5.4, J6.1, J6.2, J6.3, J6.4, J7.1, J7.2, J7.3, J7.4, J8.1, J8.2, J8.3, J8.4, MP1.1, MP2.1, MP3.1, MP4.1, S1.3; no longer D10.2, D11.2, D3.2, D4.2, D6.2, D7.2, D8.2, D9.2
- net LOAD_1: now also J4.5, J4.6, J4.7, J4.8
- net LOAD_2: now also J7.5, J7.6, J7.7, J7.8
- net LOAD_3: now also J5.5, J5.6, J5.7, J5.8
- net LOAD_4: now also J8.5, J8.6, J8.7, J8.8
- net LOAD_5: now also J6.5, J6.6, J6.7, J6.8
- net PSU_ON: now also S1.2
- net VCC3V3: now also Q11.2
- net VCC5V0: now also J1.4, J11.4, J12.4, J13.4, J14.4
- net at D5.1 (C): now also R41.1
- net at D5.2 (A): now also Q11.3; no longer R41.1
- net at R40.1: now also Q11.1
- net at R53.1: now also D8.2 (A); no longer D8.1
- net at R51.1: now also D6.2 (A); no longer D6.1
- net at R11.1: now also D3.2 (A); no longer D3.1
- net at R12.1: now also D4.2 (A); no longer D4.1
- net at R52.1: now also D7.2 (A); no longer D7.1
- net at R55.1: now also D10.2 (A); no longer D10.1
- net at R56.1: now also D11.2 (A); no longer D11.1
- net at R54.1: now also D9.2 (A); no longer D9.1
- net P3/4 renamed VCC12V0
- net VCC12V0: now also J1.1, J11.1, J12.1, J13.1, J14.1
- new net: S1.S1 (SH), S1.S2 (SH), S1.S3 (SH), S1.S4 (SH)
- no-connect marks 2 -> 5
Other:
- moved on the sheet: D12, D13, R11, R12, R40, R41, R51, R52, R53, R54, R55, R56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
